Commit message: #62: Refactored Files

File: overlay_ws/src/kr240_r2900_2/omni_urdf/kr240_r2900_2.urdf.xacro (robot description, xacro)
@@ -1,6 +1,5 @@
 <?xml version="1.0" ?>
 <robot name="kuka_with_omnimove" xmlns:xacro="http://wiki.ros.org/xacro">
-  <xacro:include filename="$(find kr240_r2900_2)/urdf/kr240_r2900_2_macro_omni.xacro"/>
-  <xacro:include filename="$(find kr240_r2900_2)/urdf/kr_quantec_ros2_control_macro.xacro"/>
+  <xacro:include filename="$(find kr240_r2900_2)/omni_urdf/kr240_r2900_2_omni.urdf.xacro"/>
   <xacro:include filename="$(find kuka_omnimove_e575_support)/urdf/omnimove.xacro"/>
   <xacro:include filename="$(find sick_safetyscanners2)/description/urdf/nanoscan3/nanoscan3_macro.xacro"/>
@@ -14,38 +13,15 @@
     <origin xyz="0 0 0" rpy="0 0 0"/>
   </joint>
-  <joint name="platform_to_arm_joint" type="fixed">
+  <joint name="base_to_platform" type="fixed">
+    <parent link="omnimove_base"/>
+    <child link="omnimove_platform"/>
+    <origin xyz="0 0 0.6" rpy="0 0 0"/>
+  </joint>
+  <!-- Attach KUKA robot to the omnimove platform -->
+  <joint name="robot_mount" type="fixed">
     <parent link="omnimove_platform"/>
     <child link="base_link"/>
     <origin xyz="0.9 0 0.85" rpy="0 0 0"/>
   </joint>
-  <!-- Read additional arguments  -->
-  <xacro:arg name="driver_version" default="rsi_only"/>
-  <xacro:arg name="mode" default="hardware"/>
-  <xacro:arg name="use_gpio" default="false"/>
-  <xacro:arg name="roundtrip_time" default="0"/>
-  <xacro:arg name="client_ip" default="0.0.0.0"/>
-  <xacro:arg name="client_port" default="59152"/>
-  <xacro:arg name="controller_ip" default="0.0.0.0"/>
-  <xacro:arg name="verify_robot_model" default="true"/>
-  <xacro:arg name="prefix" default=""/>
-  <xacro:arg name="x" default="0.9"/>   <!-- Changed from 0 -->
-  <xacro:arg name="y" default="0"/>
-  <xacro:arg name="z" default="0.85"/>  <!-- Changed from 0 -->
-  <xacro:arg name="roll" default="0"/>
-  <xacro:arg name="pitch" default="0"/>
-  <xacro:arg name="yaw" default="0"/>
-  <xacro:kuka_quantec_ros2_control name="$(arg prefix)kr240_r2900_2"
-  driver_version="$(arg driver_version)"
-  client_ip="$(arg client_ip)"
-  client_port="$(arg client_port)"
-  controller_ip="$(arg controller_ip)"
-  prefix="$(arg prefix)"
-  mode="$(arg mode)"
-  use_gpio="$(arg use_gpio)"
-  roundtrip_time="$(arg roundtrip_time)"
-  verify_robot_model="$(arg verify_robot_model)"/>
-  <xacro:kuka_kr240_r2900_2_robot prefix="$(arg prefix)" package_name="kr240_r2900_2">
-    <origin xyz="$(arg x) $(arg y) $(arg z)" rpy="$(arg roll) $(arg pitch) $(arg yaw)"/>
-  </xacro:kuka_kr240_r2900_2_robot>
   <!-- Add nanoscan3 sensors at specific locations on omnimove -->
   <!-- Front-right sensor -->

File: overlay_ws/src/kr240_r2900_2/omni_urdf/kr240_r2900_2_omni.urdf.xacro (robot description, xacro)
@@ -2,6 +2,6 @@
 <robot xmlns:xacro="http://ros.org/wiki/xacro" name="kr240_r2900_2">
   <!-- Import macro files  -->
-  <xacro:include filename="$(find kr240_r2900_2)/urdf/kr240_r2900_2_macro_omni.xacro"/>
-  <xacro:include filename="$(find kr240_r2900_2)/urdf/kr_quantec_ros2_control_macro.xacro"/>
+  <xacro:include filename="$(find kr240_r2900_2)/omni_urdf/kr240_r2900_2_macro_omni.xacro"/>
+  <xacro:include filename="$(find kr240_r2900_2)/omni_urdf/kr_quantec_ros2_control_macro.xacro"/>
   <!-- Read additional arguments  -->
   <xacro:arg name="driver_version" default="rsi_only"/>

File: overlay_ws/src/kr240_r2900_2/urdf/kr240_r2900_2.urdf.xacro (robot description, xacro)
@@ -1,22 +1,7 @@
-<?xml version="1.0" ?>
-<robot name="kuka_with_omnimove" xmlns:xacro="http://wiki.ros.org/xacro">
-  <xacro:include filename="$(find kr240_r2900_2)/urdf/kr240_r2900_2_macro_omni.xacro"/>
+<?xml version="1.0" encoding="UTF-8"?>
+<robot xmlns:xacro="http://ros.org/wiki/xacro" name="kr240_r2900_2">
+  <!-- Import macro files  -->
+  <xacro:include filename="$(find kr240_r2900_2)/urdf/kr240_r2900_2_macro.xacro"/>
   <xacro:include filename="$(find kr240_r2900_2)/urdf/kr_quantec_ros2_control_macro.xacro"/>
-  <xacro:include filename="$(find kuka_omnimove_e575_support)/urdf/omnimove.xacro"/>
-  <xacro:include filename="$(find sick_safetyscanners2)/description/urdf/nanoscan3/nanoscan3_macro.xacro"/>
-  <xacro:omnimove prefix="omnimove_"/>
-  <xacro:omnimove_ros2_control name="omnimove"/>
-  <!-- place the omnimove on the world ground plane (omnimove_base is child of world)
-       Adjust the origin's z value if the mesh is not grounded at its link frame. -->
-  <joint name="omni_to_world" type="fixed">
-    <parent link="world"/>
-    <child link="omnimove_base"/>
-    <origin xyz="0 0 0" rpy="0 0 0"/>
-  </joint>
-  <joint name="platform_to_arm_joint" type="fixed">
-    <parent link="omnimove_platform"/>
-    <child link="base_link"/>
-    <origin xyz="0.9 0 0.85" rpy="0 0 0"/>
-  </joint>
   <!-- Read additional arguments  -->
   <xacro:arg name="driver_version" default="rsi_only"/>
@@ -29,53 +14,23 @@
   <xacro:arg name="verify_robot_model" default="true"/>
   <xacro:arg name="prefix" default=""/>
-  <xacro:arg name="x" default="0.9"/>   <!-- Changed from 0 -->
+  <xacro:arg name="x" default="0"/>
   <xacro:arg name="y" default="0"/>
-  <xacro:arg name="z" default="0.85"/>  <!-- Changed from 0 -->
+  <xacro:arg name="z" default="0"/>
   <xacro:arg name="roll" default="0"/>
   <xacro:arg name="pitch" default="0"/>
   <xacro:arg name="yaw" default="0"/>
-  <xacro:kuka_quantec_ros2_control name="$(arg prefix)kr240_r2900_2"
-  driver_version="$(arg driver_version)"
-  client_ip="$(arg client_ip)"
-  client_port="$(arg client_port)"
-  controller_ip="$(arg controller_ip)"
-  prefix="$(arg prefix)"
-  mode="$(arg mode)"
-  use_gpio="$(arg use_gpio)"
-  roundtrip_time="$(arg roundtrip_time)"
-  verify_robot_model="$(arg verify_robot_model)"/>
+  <xacro:kuka_quantec_ros2_control
+          name="$(arg prefix)kr240_r2900_2"
+          driver_version="$(arg driver_version)"
+          client_ip="$(arg client_ip)"
+          client_port="$(arg client_port)"
+          controller_ip="$(arg controller_ip)"
+          prefix="$(arg prefix)"
+          mode="$(arg mode)"
+          use_gpio="$(arg use_gpio)"
+          roundtrip_time="$(arg roundtrip_time)"
+          verify_robot_model="$(arg verify_robot_model)"/>
   <xacro:kuka_kr240_r2900_2_robot prefix="$(arg prefix)" package_name="kr240_r2900_2">
     <origin xyz="$(arg x) $(arg y) $(arg z)" rpy="$(arg roll) $(arg pitch) $(arg yaw)"/>
   </xacro:kuka_kr240_r2900_2_robot>
-  <!-- Add nanoscan3 sensors at specific locations on omnimove -->
-  <!-- Front-right sensor -->
-  <xacro:nanoscan3
-    name="nanoscan3_front_right"
-    parent="omnimove_platform"
-    mounting_kit="true"
-    ros_topic="/nanoscan3_front_right"
-    update_rate="50.0"
-    min_angle="${radians(-45)}"
-    max_angle="${radians(225)}"
-    min_range="0.05"
-    max_range="10.0"
-    gaussian_noise="0.006"
-    max_beams="500">
-    <origin xyz="1.55 -0.925 0.175" rpy="0 0 ${radians(-45)}" />
-  </xacro:nanoscan3>
-  <!-- Back-Left sensor -->
-  <xacro:nanoscan3
-    name="nanoscan3_back_left"
-    parent="omnimove_platform"
-    mounting_kit="true"
-    ros_topic="/nanoscan3_back_left"
-    update_rate="50.0"
-    min_angle="${radians(-45)}"
-    max_angle="${radians(225)}"
-    min_range="0.05"
-    max_range="10.0"
-    gaussian_noise="0.006"
-    max_beams="500">
-    <origin xyz="-1.55 0.925 0.175" rpy="0 0 ${radians(135)}" />
-  </xacro:nanoscan3>
 </robot>

Commit message: #68: Updated file permissions

File: overlay_ws/src/kr240_r2900_2/omni_urdf/kr240_r2900_2.urdf.xacro (robot description, xacro)
@@ -8,13 +8,8 @@
   <!-- place the omnimove on the world ground plane (omnimove_base is child of world)
        Adjust the origin's z value if the mesh is not grounded at its link frame. -->
-  <joint name="omni_to_world" type="fixed">
-    <parent link="world"/>
-    <child link="omnimove_base"/>
-    <origin xyz="0 0 0" rpy="0 0 0"/>
-  </joint>
   <joint name="base_to_platform" type="fixed">
     <parent link="omnimove_base"/>
     <child link="omnimove_platform"/>
-    <origin xyz="0 0 0.6" rpy="0 0 0"/>
+    <origin xyz="0 0 0" rpy="0 0 0"/>
   </joint>
   <!-- Attach KUKA robot to the omnimove platform -->

File: overlay_ws/src/kr240_r2900_2/omni_urdf/kr240_r2900_2_macro_omni.xacro (robot description, xacro)
@@ -138,5 +138,5 @@
     </link>
     <link name="${prefix}tool0"/>
-    <link name="world"/>
+    <!-- <link name="world"/> -->
     <joint name="${prefix}base_link-base" type="fixed">
       <child link="${prefix}base"/>

File: overlay_ws/src/kuka_omnimove_e575_support/urdf/omnimove.xacro (robot description, xacro)
@@ -9,5 +9,5 @@
       </link>
       <!-- X axis prismatic joint -->
-      <joint name="${prefix}x_joint" type="prismatic">
+      <!-- <joint name="${prefix}x_joint" type="prismatic">
         <parent link="${prefix}base"/>
         <child link="${prefix}x_link"/>
@@ -19,7 +19,7 @@
           <inertia ixx="0.001" ixy="0.0" ixz="0.0" iyy="0.001" iyz="0.0" izz="0.001"/>
         </inertial>
-      </link>
+      </link> -->
       <!-- Y axis prismatic joint -->
-      <joint name="${prefix}y_joint" type="prismatic">
+      <!-- <joint name="${prefix}y_joint" type="prismatic">
         <parent link="${prefix}x_link"/>
         <child link="${prefix}y_link"/>
@@ -32,12 +32,12 @@
           <inertia ixx="0.001" ixy="0.0" ixz="0.0" iyy="0.001" iyz="0.0" izz="0.001"/>
         </inertial>
-      </link>
+      </link> -->
       <!-- Z axis rotational joint (rotation) -->
-      <joint name="${prefix}z_joint" type="revolute">
+      <!-- <joint name="${prefix}z_joint" type="revolute">
         <parent link="${prefix}y_link"/>
         <child link="${prefix}platform"/>
         <axis xyz="0 0 1"/>
         <limit lower="-3.14159" upper="3.14159" effort="1000" velocity="1.0"/>
-      </joint>
+      </joint> -->
       <link name="${prefix}platform">
         <visual>
