Commit message: #70: Add scanner documentation, update URDF macros, and enhance motion planning

File: overlay_ws/src/kr240_r2900_2/omni_urdf/kr240_r2900_2_macro_omni.xacro (robot description, xacro)
@@ -3,5 +3,5 @@
   <xacro:macro name="kuka_kr240_r2900_2_robot" params="prefix package_name *origin">
     <link name="${prefix}base"/>
-    <link name="${prefix}base_link">
+    <link name="${prefix}arm_base_link">
       <collision>
         <geometry>
@@ -139,7 +139,7 @@
     <link name="${prefix}tool0"/>
     <!-- <link name="world"/> -->
-    <joint name="${prefix}base_link-base" type="fixed">
+    <joint name="${prefix}arm_base_link-base" type="fixed">
       <child link="${prefix}base"/>
-      <parent link="${prefix}base_link"/>
+      <parent link="${prefix}arm_base_link"/>
     </joint>
     <joint name="${prefix}joint_1" type="revolute">
@@ -148,5 +148,5 @@
       <limit effort="7.29E3" lower="-3.2288591125E0" upper="3.2288591125E0" velocity="1.7976891295541595E0"/>
       <origin rpy="3.141592653589793 -0.0 0.0" xyz="0.0 0.0 0.30560000000000004"/>
-      <parent link="${prefix}base_link"/>
+      <parent link="${prefix}arm_base_link"/>
     </joint>
     <joint name="${prefix}joint_2" type="revolute">

File: overlay_ws/src/kuka_omnimove_e575_support/urdf/omnimove.xacro (robot description, xacro)
@@ -58,5 +58,5 @@
 	    <ros2_control name="omnimove" type="system">
             <hardware>
-                <plugin>kuka_mock_hardware_interface::KukaMockHardwareInterface</plugin> <!-- Changed from omnimove::KukaUTV3HardwareInterface -->
+                <plugin>omnimove::KukaUTV3HardwareInterface</plugin> <!-- Changed from omnimove::KukaUTV3HardwareInterface -->
                 <param name ="host">127.0.0.1</param>
                 <param name="port">24000</param>
